File: v2/hardware/meshbot_kicad/meshbot_kicad.kicad_pcb (KiCad board)
At the start: 2 copper layers, 88 x 72.7 mm, 39 parts, among them J1 Conn_01x02_Socket, J10 Micro_SD_Card, J11 Conn_01x03_Pin, J12 Conn_01x06_Socket, J2 Conn_01x04_Pin, J3 Conn_01x04_Pin, J4 Conn_01x01_Socket, J5 Conn_01x04_Pin, J6 Screw_Terminal_01x04, J7 Screw_Terminal_01x03, J8 Conn_01x03_Socket, J9 Conn_01x02_Socket, SW1 SW_Push, SW2 SW_Push, SW3 SW_Push, SW4 SW_Push, SW5 SW_Push, SW6 SW_Push, SW7 SW_Push, SW8 SW_Push, U1 wio-sx1262, U2 nice_nano_clean, U3 nice_nano_clean, U4 grove_a, U5 grove_a

Commit message: update
Parts:
- moved R7 1.90 mm to (158.2, 43.0), turned to -90 degrees
Routing:
- net GND: track 390.3 -> 461.4 mm, vias 38 -> 45
- net BAT: track 171.6 -> 210.8 mm, vias 12 -> 16
- net SCK:C: track 0.00 -> 38.3 mm, vias 0 -> 3
- net Net-(D2-A): track 0.00 -> 36.9 mm, vias 0 -> 2
- net 3V3: track 296.8 -> 325.7 mm, vias 19 -> 24
- net SD_CS: track 54.2 -> 26.3 mm, vias 5 -> 2
- net MISO:C: track 0.00 -> 26.4 mm, vias 0 -> 3
- net LED_B: track 1.73 -> 27.6 mm, vias 0 -> 1
- net MOSI:C: track 0.00 -> 25.6 mm, vias 0 -> 3
- net SDA: track 69.7 -> 90.2 mm, vias 3 -> 5
- net V_EXT: track 42.2 -> 62.2 mm, vias 3 -> 4
- net LED_A: track 0.60 -> 20.4 mm, vias 0 -> 2
- net Net-(D1-A): track 15.6 -> 3.98 mm
- net BUTTON_B: track 42.7 -> 51.5 mm, vias 3 -> 1
- net BUTTON_C: track 58.5 -> 64.7 mm
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Other:
- board text added: "MESHBOT version 2"
- board text added: "v2"
- board text removed: "MESHBOT version 1"
- board text removed: "v1"
